Commit message: latest updates

File: tracked_robot_description/urdf/tracked_robot.urdf (robot description, URDF)
Before this commit: robot tracked_robot, 2 links, 1 joints
Links:
- added link base_footprint
- added link left_wheel, mass 1.0; collision cylinder length=0.05 radius=0.08; visual cylinder length=0.05 radius=0.08
- added link right_wheel, mass 1.0; collision cylinder length=0.05 radius=0.08; visual cylinder length=0.05 radius=0.08
- link zed2i_camera_center: mass None -> 0.1
Joints:
- added joint base_footprint_joint: type fixed, parent base_footprint, child base_link, origin xyz=0 0 0.05 rpy=0 0 0
- added joint left_wheel_joint: type continuous, parent base_link, child left_wheel, origin xyz=0.0 0.2 0.0 rpy=1.5708 0 0, axis 0 0 -1
- added joint right_wheel_joint: type continuous, parent base_link, child right_wheel, origin xyz=0.0 -0.2 0.0 rpy=1.5708 0 0, axis 0 0 -1
